File: perfboard_x1.kicad_sch (KiCad schematic)
At the start: 120 parts, among them J1 Conn_01x10, J10 Conn_01x10, J100 Conn_01x10, J101 Conn_01x10, J102 Conn_01x10, J103 Conn_01x10, J104 Conn_01x10, J105 Conn_01x10, J106 Conn_01x10, J107 Conn_01x10, J108 Conn_01x10, J109 Conn_01x10, J11 Conn_01x10, J110 Conn_01x10, J111 Conn_01x10, J112 Conn_01x10, J113 Conn_01x10, J114 Conn_01x10, J115 Conn_01x10, J116 Conn_01x10, J117 Conn_01x10, J118 Conn_01x10, J119 Conn_01x10, J12 Conn_01x10, J120 Conn_01x10, J13 Conn_01x10, J14 Conn_01x10, J15 Conn_01x10, J16 Conn_01x10, J17 Conn_01x10, J18 Conn_01x10, J19 Conn_01x10, J2 Conn_01x10, J20 Conn_01x10, J21 Conn_01x10, J22 Conn_01x10, J23 Conn_01x10, J24 Conn_01x10, J25 Conn_01x10, J26 Conn_01x10, J27 Conn_01x10, J28 Conn_01x10, J29 Conn_01x10, J3 Conn_01x10, J30 Conn_01x10, J31 Conn_01x10, J32 Conn_01x10, J33 Conn_01x10, J34 Conn_01x10, J35 Conn_01x10, J36 Conn_01x10, J37 Conn_01x10, J38 Conn_01x10, J39 Conn_01x10, J4 Conn_01x10, J40 Conn_01x10, J41 Conn_01x10, J42 Conn_01x10, J43 Conn_01x10, J44 Conn_01x10, J45 Conn_01x10, J46 Conn_01x10, J47 Conn_01x10, J48 Conn_01x10, J49 Conn_01x10, J5 Conn_01x10, J50 Conn_01x10, J51 Conn_01x10, J52 Conn_01x10, J53 Conn_01x10, J54 Conn_01x10, J55 Conn_01x10, J56 Conn_01x10, J57 Conn_01x10, J58 Conn_01x10, J59 Conn_01x10, J6 Conn_01x10, J60 Conn_01x10, J61 Conn_01x10, J62 Conn_01x10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

Commit message: Added a sample circuit
Parts:
- added C1, C2, C3: C, Capacitor_SMD:C_1206_3216Metric, symbol Device:C
- added Q1: S8050_smd, aadhunix:SOT-23_alternate_handsoldering, symbol aadhunix:S8050_smd
- added R1, R2, R3, R4: R, Resistor_SMD:R_1206_3216Metric, symbol Device:R
- J1, J10, J100, J101, J102, J103, J104, J105, J106, J107, J108, J109, J11, J110, J111, J112, J113, J114, J115, J116, J117, J118, J119, J12, J120, J13, J14, J15, J16, J17, J18, J19, J2, J20, J21, J22, J23, J24, J25, J26, J27, J28, J29, J3, J30, J31, J32, J33, J34, J35, J36, J37, J38, J39, J4, J40, J41, J42, J43, J44, J45, J46, J47, J48, J49, J5, J50, J51, J52, J53, J54, J55, J56, J57, J58, J59, J6, J60, J61, J62, J63, J64, J65, J66, J67, J68, J69, J7, J70, J71, J72, J73, J74, J75, J76, J77, J78, J79, J8, J80, J81, J82, J83, J84, J85, J86, J87, J88, J89, J9, J90, J91, J92, J93, J94, J95, J96, J97, J98, J99: now left out of the parts list
Connections:
- new net: C3.1, Q1.3 (C), R3.2
- new net: C2.2, Q1.1 (B), R1.2, R2.1
- new net: C1.1, Q1.2 (E), R4.1
- new net GND: C1.2, R2.2, R4.2
- new net VCC: R1.1, R3.1
Other:
- moved on the sheet: J1, J10, J100, J101, J102, J103, J104, J105, J106, J107, J108, J109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
